File: Hardware/PUTM_EV_CART_INDICATOR.kicad_pcb (KiCad board)
At the start: 2 copper layers, 39.5 x 16 mm, 11 parts, among them J3 Screw_Terminal_01x06, Q2 2N7002, Q3 2N7002

Commit message: update
Parts:
- removed REF** (x2): MountingHole_2.2mm_M2, MountingHole:MountingHole_2.2mm_M2
- added H1: MountingHole, MountingHole:MountingHole_2.2mm_M2, F.Cu at (81.0, 78.5)
- added H2: MountingHole, MountingHole:MountingHole_2.2mm_M2, F.Cu at (81.0, 85.4)
- Q2, Q3: value 2N7002 -> ~
- R8: value 2.2k -> 1.1k
- moved Q2 1.04 mm to (105.5, 86.9)
Connections:
- D3 pad 2: Net-(D3-A) -> /IMD_LED
- J3 pad 6: unconnected-(J3-Pin_6-Pad6) -> /IMD_LED
- Q2 pad 3: Net-(D3-A) -> /IMD_LED
- R8 pad 1: Net-(D3-A) -> /IMD_LED
Routing:
- net /IMD_LED: track 0.00 -> 16.4 mm
- net Net-(D3-A): track 7.75 -> 0.00 mm
- net /IMD: track 9.64 -> 8.61 mm

Commit message: poprawy
Parts:
- removed J3: Screw_Terminal_01x06, Include:TB00250006BE
- added J1: Screw_Terminal_01x08, Include:TB00150008BE, F.Cu at (85.5, 73.5)
- added K1: IMB03ITS, Include:IMB03ITS, F.Cu at (94.6, 88.1)
- added K2: IMB03ITS, Include:IMB03ITS, F.Cu at (112.1, 87.7)
- added R9: 2.2k, Resistor_SMD:R_0603_1608Metric_Pad0.98x0.95mm_HandSolder, F.Cu at (100.2, 86.7)
- moved H1 18.5 mm to (66.5, 90.0)
- moved H2 10.7 mm to (71.0, 81.5)
- moved D2 4.46 mm to (99.5, 83.3)
- moved D3 4.46 mm to (111.2, 83.7)
- moved Q2 4.46 mm to (106.7, 82.6)
- moved R7 4.46 mm to (96.1, 83.3)
- moved R8 4.46 mm to (114.8, 83.9)
- moved Q3 4.46 mm to (91.9, 83.2)
- moved R21 4.46 mm to (103.6, 82.7)
- moved R4 4.46 mm to (87.8, 83.4)
Connections:
- net /bulb_ground renamed Net-(K1-COIL_1)
Routing:
- net +24V: track 49.2 -> 92.9 mm
- net /TSAL_LED: track 0.00 -> 16.9 mm
- net Net-(K1-COIL_1): track 27.0 -> 17.3 mm
- net /bulb_imd+: track 0.00 -> 8.33 mm
- net /TSAL_GREEN: track 13.8 -> 20.8 mm
- net /IMD_LED: track 16.4 -> 22.7 mm, vias 0 -> 1
- net /IMD: track 8.61 -> 12.1 mm, vias 0 -> 1
- net /bulb+: track 0.00 -> 1.42 mm
- net GND: vias 7 -> 6
- removed copper zone on B.Cu, net GND
- removed copper zone on F.Cu, net GND
Other:
- board size 39.5 x 16 mm -> 46 x 34.5 mm

Commit message: Zmieniono na przekaźniki
Parts:
- removed K1, K2: IMB03ITS, Include:IMB03ITS
- removed Q2, Q3: ~, Package_TO_SOT_SMD:SOT-23
- removed R21, R4: 10k, Resistor_SMD:R_0603_1608Metric_Pad0.98x0.95mm_HandSolder
- removed R7, R9: 2.2k, Resistor_SMD:R_0603_1608Metric_Pad0.98x0.95mm_HandSolder
- added D1: D, Diode_SMD:D_0603_1608Metric_Pad1.05x0.95mm_HandSolder, F.Cu at (107.0, 81.6)
- added D4: LED, LED_SMD:LED_0603_1608Metric, F.Cu at (120.9, 80.0)
- added K3: IM07DTS, Include:IM23TS, F.Cu at (101.9, 77.5)
- added K4: IM07DTS, Include:IM23TS, F.Cu at (111.9, 77.5)
- added Q4: ~, Package_TO_SOT_SMD:SOT-23, F.Cu at (118.9, 74.0)
- added Q5: ~, Package_TO_SOT_SMD:SOT-23, F.Cu at (95.0, 74.0)
- added R10: 100, Resistor_SMD:R_0603_1608Metric_Pad0.98x0.95mm_HandSolder, F.Cu at (123.0, 75.0)
- added R11: 1K, Resistor_SMD:R_0603_1608Metric_Pad0.98x0.95mm_HandSolder, F.Cu at (117.4, 80.0)
- added R12: 1K, Resistor_SMD:R_0603_1608Metric_Pad0.98x0.95mm_HandSolder, F.Cu at (96.4, 78.1)
- added R22: 10k, Resistor_SMD:R_0603_1608Metric_Pad0.98x0.95mm_HandSolder, F.Cu at (122.9, 73.0)
- added R6: 100, Resistor_SMD:R_0603_1608Metric_Pad0.98x0.95mm_HandSolder, F.Cu at (90.9, 73.0)
- D2: value LED -> D; footprint LED_SMD:LED_0603_1608Metric -> Diode_SMD:D_0603_1608Metric_Pad1.05x0.95mm_HandSolder
- R8: value 1.1k -> 10k
- moved R8 25.5 mm to (90.9, 75.0), turned to 180 degrees
- moved H1 20.6 mm to (85.0, 81.0)
- moved D3 18.9 mm to (92.5, 81.0)
- moved H2 15.9 mm to (85.0, 74.0)
- moved D2 10.5 mm to (107.0, 76.0), turned to 90 degrees
- moved J1 8.24 mm to (86.0, 65.3)
Connections:
- D2 pad 1: Net-(D2-K) -> +24V
- D2 pad 2: +24V -> Net-(D2-A)
- D3 pad 2: /IMD_LED -> /TSAL_LED
- J1 pad 1: +24V -> /TSAL_COLUMN
- J1 pad 2: GND -> /TSAL_LED
- J1 pad 4: /IMD -> +24V
- J1 pad 5: /bulb+ -> GND
- J1 pad 6: /IMD_LED -> /IMD
- J1 pad 7: /TSAL_LED -> /IMD_LED
- J1 pad 8: /bulb_imd+ -> /IMD_COLUMN
- R8 pad 1: /IMD_LED -> GND
- R8 pad 2: +24V -> Net-(Q5-G)
Routing:
- net +24V: track 92.9 -> 49.4 mm
- net /TSAL_COLUMN: track 0.00 -> 33.5 mm
- net /IMD_COLUMN: track 0.00 -> 18.8 mm
- net /IMD: track 12.1 -> 30.4 mm, vias 1 -> 0
- net Net-(K1-COIL_1): track 17.3 -> 0.00 mm
- net Net-(D1-A): track 0.00 -> 16.0 mm, vias 0 -> 1
- net Net-(D2-A): track 0.00 -> 13.0 mm
- net Net-(K4-NC_2): track 0.00 -> 11.0 mm
- net /TSAL_GREEN: track 20.8 -> 10.2 mm
- net /bulb_imd+: track 8.33 -> 0.00 mm
- net /TSAL_LED: track 16.9 -> 24.6 mm
- net /IMD_LED: track 22.7 -> 17.7 mm, vias 1 -> 0
- net Net-(Q5-G): track 0.00 -> 4.99 mm
- net Net-(Q4-G): track 0.00 -> 4.98 mm
- net Net-(K3-NO_1): track 0.00 -> 3.87 mm
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- added copper zone on B.Cu, net GND
- added copper zone on F.Cu, net GND
Other:
- board size 46 x 34.5 mm -> 43 x 25 mm
- board text added: "{dblquote}Nie czarodziejska tylko magiczna i nie fujarka tylko flet... magiczna flet{dblquote} ~Ojciec Franz Pijo"
