File: Hardware/PUTM_EV_CART_INDICATOR.kicad_sch (KiCad schematic)
At the start: 9 parts, among them J3 Screw_Terminal_01x06

Commit message: Zaktualizowano do standarow PUTM
Other:
- note removed: "Outside of PCB"
Changed lines of the file:
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@@
-		)
-	)
-	(text "Outside \nof\nPCB\n"
-		(exclude_from_sim no)
-		(at 133.35 19.05 0)
-		(effects
-			(font
-				(size 1.27 1.27)
-			)
 		)
 	)

Commit message: update
Parts:
- added H1, H2: MountingHole, MountingHole:MountingHole_2.2mm_M2, symbol Mechanical:MountingHole
- R8: value 2.2k -> 1.1k
Connections:
- net IMD_LED: now reaches D3.2 (A), Q2.3 (D), R8.1
- net IMD_LED: now also J3.6 (Pin_6)
- no-connect marks 1 -> 0
Changed lines of the file:
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@@
 		(color 0 0 0 0)
 	)
-	(no_connect
-		(at 33.02 33.02)
-	)
 	(wire
 		(pts
@@
 	(wire
 		(pts
+			(xy 80.01 52.07) (xy 67.31 52.07)
+		)
+		(stroke
+			(width 0)
+			(type default)
+		)
+	)
+	(wire
+		(pts
 			(xy 133.35 49.53) (xy 149.86 49.53)
 		)
@@
 	(wire
 		(pts
+			(xy 80.01 55.88) (xy 80.01 52.07)
+		)
+		(stroke
+			(width 0)
+			(type default)
+		)
+	)
+	(wire
+		(pts
 			(xy 67.31 52.07) (xy 67.31 53.34)
 		)
@@
 	(wire
 		(pts
+			(xy 33.02 33.02) (xy 39.37 33.02)
+		)
+		(stroke
+			(width 0)
+			(type default)
+		)
+	)
+	(wire
+		(pts
 			(xy 149.86 34.29) (xy 149.86 35.56)
 		)
@@
 			(width 0)
 			(type default)
+		)
+	)
+	(label "IMD_LED"
+		(at 39.37 33.02 0)
+		(effects
+			(font
+				(size 1.27 1.27)
+			)
+			(justify left bottom)
 		)
 	)
@@
 		)
 	)
+	(label "IMD_LED"
+		(at 80.01 55.88 270)
+		(effects
+			(font
+				(size 1.27 1.27)
+			)
+			(justify right bottom)
+		)
+	)
 	(label "TSAL_GREEN"
 		(at 39.37 25.4 0)
@@
 	)
 	(symbol
+		(lib_id "Mechanical:MountingHole")
+		(at 265.43 17.78 0)
+		(unit 1)
+		(exclude_from_sim no)
+		(in_bom no)
+		(on_board yes)
+		(dnp no)
+		(fields_autoplaced yes)
+		(property "Reference" "H1"
+			(at 267.97 16.5099 0)
+			(effects
+				(font
+					(size 1.27 1.27)
+				)
+				(justify left)
+			)
+		)
+		(property "Value" "MountingHole"
+			(at 267.97 19.0499 0)
+			(effects
+				(font
+					(size 1.27 1.27)
+				)
+				(justify left)
+			)
+		)
+		(property "Footprint" "MountingHole:MountingHole_2.2mm_M2"
+			(at 265.43 17.78 0)
+			(effects
+				(font
+					(size 1.27 1.27)
+				)
+				(hide yes)
+			)
+		)
+		(property "Datasheet" "~"
+			(at 265.43 17.78 0)
+			(effects
+				(font
+					(size 1.27 1.27)
+				)
+				(hide yes)
+			)
+		)
+		(property "Description" "Mounting Hole without connection"
+			(at 265.43 17.78 0)
+			(effects
+				(font
+					(size 1.27 1.27)
+				)
+				(hide yes)
+			)
+		)
+		(instances
+			(project ""
+				(path "/273ec47a-aafc-4766-bd44-1878375efcdd"
+					(reference "H1")
+					(unit 1)
+				)
+			)
+		)
+	)
+	(symbol
 		(lib_id "Device:R_Small")
 		(at 120.65 59.69 0)
@@
 			)
 		)
-		(property "Value" "2.2k"
+		(property "Value" "1.1k"
 			(at 69.85 49.53 0)
 			(effects
@@
 					(unit 1)
 				)
+			)
+		)
+	)
+	(symbol
+		(lib_id "Mechanical:MountingHole")
+		(at 265.43 26.67 0)
+		(unit 1)
+		(exclude_from_sim no)
+		(in_bom no)
+		(on_board yes)
+		(dnp no)
+		(fields_autoplaced yes)
+		(property "Reference" "H2"
+			(at 267.97 25.3999 0)
+			(effects
+				(font
+					(size 1.27 1.27)
+				)
+				(justify left)
+			)
+		)
+		(property "Value" "MountingHole"
+			(at 267.97 27.9399 0)
+			(effects
+				(font
+					(size 1.27 1.27)
+				)
+				(justify left)
+			)
+		)
+		(property "Footprint" "MountingHole:MountingHole_2.2mm_M2"
+			(at 265.43 26.67 0)
+			(effects
+				(font
+					(size 1.27 1.27)
+				)
+				(hide yes)
+			)
+		)
+		(property "Datasheet" "~"
+			(at 265.43 26.67 0)
+			(effects
+				(font
+					(size 1.27 1.27)
+				)
+				(hide yes)
+			)
+		)
+		(property "Description" "Mounting Hole without connection"
+			(at 265.43 26.67 0)
+			(effects
+				(font
+					(size 1.27 1.27)
+				)
+				(hide yes)
+			)
+		)
+		(instances
+			(project "PUTM_EV_CART_INDICATOR"
+				(path "/273ec47a-aafc-4766-bd44-1878375efcdd"
+					(reference "H2")
+					(unit 1)
+				)

Commit message: poprawy
Parts:
- removed D2: LED, LED_SMD:LED_0603_1608Metric, symbol Device:LED
- removed J3: Screw_Terminal_01x06, Include:TB00250006BE, symbol Connector:Screw_Terminal_01x06
- removed Q2, Q3: ~, Package_TO_SOT_SMD:SOT-23, symbol PUTM_EV_IMD_SAFETY_2021-rescue:2N7002-Transistor_FET
- removed R21, R4: 10k, Resistor_SMD:R_0603_1608Metric_Pad0.98x0.95mm_HandSolder, symbol Device:R_Small
- removed R7: 2.2k, Resistor_SMD:R_0603_1608Metric_Pad0.98x0.95mm_HandSolder, symbol Device:R_Small
- added D4: LED, LED_SMD:LED_0603_1608Metric, symbol Device:LED
- added J1: Screw_Terminal_01x08, Include:TB00150008BE, symbol Connector:Screw_Terminal_01x08
- added K3, K4: IM07DTS, Include:IM23TS, symbol Samacsys_kicad_sym:IM07DTS
- added Q4, Q5: ~, Package_TO_SOT_SMD:SOT-23, symbol PUTM_EV_IMD_SAFETY_2021-rescue:2N7002-Transistor_FET
- added R10, R6: 100, Resistor_SMD:R_0603_1608Metric_Pad0.98x0.95mm_HandSolder, symbol Device:R_Small
- added R11, R12: 1K, Resistor_SMD:R_0603_1608Metric_Pad0.98x0.95mm_HandSolder, symbol Device:R_Small
- added R22: 10k, Resistor_SMD:R_0603_1608Metric_Pad0.98x0.95mm_HandSolder, symbol Device:R_Small
- R8: value 1.1k -> 10k
Connections:
- net +24V: now also J1.1 (Pin_1), K3.1 (COIL_1), K3.3 (COM_1), K3.6 (COM_2), K4.1 (COIL_1), K4.3 (COM_1), K4.6 (COM_2); no longer R8.2
- net GND: now also R8.1, D4.1 (K), J1.2 (Pin_2), Q4.2 (S), Q5.2 (S), R22.2
- net IMD: now also J1.4 (Pin_4), R10.2
- net IMD_LED: now also D4.2 (A), J1.6 (Pin_6), R11.1; no longer D3.2 (A), R8.1
- net TSAL_GREEN: now also J1.3 (Pin_3), R6.2
- new net: Q4.1 (G), R10.1, R22.1
- new net: K4.8 (COIL_2), Q4.3 (D)
- new net: Q5.1 (G), R6.1, R8.2
- new net: K3.8 (COIL_2), Q5.3 (D)
- new net: K4.7 (NC_2), R11.2
- new net: K3.4 (NO_1), R12.2
- new net IMD_COLUMN: J1.8 (Pin_8), K4.2 (NC_1)
- new net TSAL_COLUMN: J1.5 (Pin_5), K3.5 (NO_2)
- new net TSAL_LED: D3.2 (A), J1.7 (Pin_7), R12.1

Commit message: Zmieniono na przekaźniki
Parts:
- added D1, D2: D, Diode_SMD:D_0603_1608Metric_Pad1.05x0.95mm_HandSolder, symbol Device:D
Connections:
- net +24V: now also J1.4 (Pin_4), D1.1 (K), D2.1 (K); no longer J1.1 (Pin_1)
- net GND: now also J1.5 (Pin_5); no longer J1.2 (Pin_2)
- net IMD: now also J1.6 (Pin_6); no longer J1.4 (Pin_4)
- net IMD_LED: now also J1.7 (Pin_7); no longer J1.6 (Pin_6)
- net TSAL_COLUMN: now also J1.1 (Pin_1); no longer J1.5 (Pin_5)
- net TSAL_LED: now also J1.2 (Pin_2); no longer J1.7 (Pin_7)
- net at K4.8 (COIL_2), Q4.3 (D): now also D1.2 (A)
- net at K3.8 (COIL_2), Q5.3 (D): now also D2.2 (A)
Other:
- moved on the sheet: J1
